Commit message: wip

File: urdf/gripper.ros2_control.xacro (robot description, xacro)
@@ -3,5 +3,5 @@
   <xacro:macro name="gripper_ros2_control" params="
     use_fake_hardware">
-<ros2_control name="RRBotGripper" type="system">
+<ros2_control name="ElectricGripper" type="actuator">
  <hardware>
    <plugin>mock_components/GenericSystem</plugin>
@@ -12,5 +12,7 @@
      <param name="max">50</param>
    </command_interface>
-   <state_interface name="position"/>
+        <state_interface name="position">
+          <param name="initial_value">0</param>
+        </state_interface>
    <!-- <state_interface name="velocity"/> -->
  </joint>

File: urdf/mycobot_320.srdf.xacro (robot description, xacro)
@@ -1,4 +1,4 @@
 <?xml version="1.0" encoding="UTF-8"?>
-<robot xmlns:xacro="http://wiki.ros.org/xacro" name="mycobot_320">
+<robot xmlns:xacro="http://wiki.ros.org/xacro" name="$(arg name)">
     <group name="arm_group">
         <joint name="joint1" />
@@ -8,4 +8,5 @@
         <joint name="joint5" />
         <joint name="joint6" />
+        <joint name="gripper_controller" />
     </group>
     <group name="gripper_group">
@@ -19,7 +20,8 @@
         <joint name="joint5" value="0" />
         <joint name="joint6" value="0" />
+        <joint name="gripper_controller" value="0" />
     </group_state>
     <virtual_joint name="vitual_joint" type="fixed" parent_frame="basic" child_link="base_link" />
-    <disable_collisions link1="base_link" link2="link1" reason="Adjacent" />
+<!--     <disable_collisions link1="base_link" link2="link1" reason="Adjacent" />
     <disable_collisions link1="base_link" link2="link4" reason="Never" />
     <disable_collisions link1="link1" link2="link2" reason="Adjacent" />
@@ -30,4 +32,81 @@
     <disable_collisions link1="link4" link2="link5" reason="Adjacent" />
     <disable_collisions link1="link4" link2="link6" reason="Never" />
-    <disable_collisions link1="link5" link2="link6" reason="Adjacent" />
+    <disable_collisions link1="link5" link2="link6" reason="Adjacent" /> -->
+    <disable_collisions link1="base_link" link2="gripper_left1" reason="Never"/>
+    <disable_collisions link1="base_link" link2="gripper_left2" reason="Never"/>
+    <disable_collisions link1="base_link" link2="gripper_left3" reason="Never"/>
+    <disable_collisions link1="base_link" link2="gripper_right1" reason="Never"/>
+    <disable_collisions link1="base_link" link2="gripper_right2" reason="Never"/>
+    <disable_collisions link1="base_link" link2="gripper_right3" reason="Never"/>
+    <disable_collisions link1="base_link" link2="link1" reason="Adjacent"/>
+    <disable_collisions link1="gripper_base" link2="gripper_left1" reason="Never"/>
+    <disable_collisions link1="gripper_base" link2="gripper_left2" reason="Adjacent"/>
+    <disable_collisions link1="gripper_base" link2="gripper_left3" reason="Adjacent"/>
+    <disable_collisions link1="gripper_base" link2="gripper_right1" reason="Never"/>
+    <disable_collisions link1="gripper_base" link2="gripper_right2" reason="Adjacent"/>
+    <disable_collisions link1="gripper_base" link2="gripper_right3" reason="Adjacent"/>
+    <disable_collisions link1="gripper_base" link2="link4" reason="Never"/>
+    <disable_collisions link1="gripper_base" link2="link5" reason="Never"/>
+    <disable_collisions link1="gripper_base" link2="link6" reason="Adjacent"/>
+    <disable_collisions link1="gripper_left1" link2="gripper_left2" reason="Default"/>
+    <disable_collisions link1="gripper_left1" link2="gripper_left3" reason="Adjacent"/>
+    <disable_collisions link1="gripper_left1" link2="gripper_right1" reason="Never"/>
+    <disable_collisions link1="gripper_left1" link2="gripper_right2" reason="Never"/>
+    <disable_collisions link1="gripper_left1" link2="gripper_right3" reason="Never"/>
+    <disable_collisions link1="gripper_left1" link2="link1" reason="Never"/>
+    <disable_collisions link1="gripper_left1" link2="link2" reason="Never"/>
+    <disable_collisions link1="gripper_left1" link2="link3" reason="Never"/>
+    <disable_collisions link1="gripper_left1" link2="link4" reason="Never"/>
+    <disable_collisions link1="gripper_left1" link2="link5" reason="Never"/>
+    <disable_collisions link1="gripper_left1" link2="link6" reason="Never"/>
+    <disable_collisions link1="gripper_left2" link2="gripper_left3" reason="Never"/>
+    <disable_collisions link1="gripper_left2" link2="gripper_right1" reason="Never"/>
+    <disable_collisions link1="gripper_left2" link2="gripper_right2" reason="Never"/>
+    <disable_collisions link1="gripper_left2" link2="gripper_right3" reason="Never"/>
+    <disable_collisions link1="gripper_left2" link2="link1" reason="Never"/>
+    <disable_collisions link1="gripper_left2" link2="link2" reason="Never"/>
+    <disable_collisions link1="gripper_left2" link2="link3" reason="Never"/>
+    <disable_collisions link1="gripper_left2" link2="link4" reason="Never"/>
+    <disable_collisions link1="gripper_left2" link2="link5" reason="Never"/>
+    <disable_collisions link1="gripper_left2" link2="link6" reason="Never"/>
+    <disable_collisions link1="gripper_left3" link2="gripper_right1" reason="Never"/>
+    <disable_collisions link1="gripper_left3" link2="gripper_right2" reason="Never"/>
+    <disable_collisions link1="gripper_left3" link2="gripper_right3" reason="Default"/>
+    <disable_collisions link1="gripper_left3" link2="link1" reason="Never"/>
+    <disable_collisions link1="gripper_left3" link2="link2" reason="Never"/>
+    <disable_collisions link1="gripper_left3" link2="link3" reason="Never"/>
+    <disable_collisions link1="gripper_left3" link2="link4" reason="Never"/>
+    <disable_collisions link1="gripper_left3" link2="link5" reason="Never"/>
+    <disable_collisions link1="gripper_left3" link2="link6" reason="Never"/>
+    <disable_collisions link1="gripper_right1" link2="gripper_right2" reason="Default"/>
+    <disable_collisions link1="gripper_right1" link2="gripper_right3" reason="Adjacent"/>
+    <disable_collisions link1="gripper_right1" link2="link1" reason="Never"/>
+    <disable_collisions link1="gripper_right1" link2="link2" reason="Never"/>
+    <disable_collisions link1="gripper_right1" link2="link3" reason="Never"/>
+    <disable_collisions link1="gripper_right1" link2="link4" reason="Never"/>
+    <disable_collisions link1="gripper_right1" link2="link5" reason="Never"/>
+    <disable_collisions link1="gripper_right1" link2="link6" reason="Never"/>
+    <disable_collisions link1="gripper_right2" link2="gripper_right3" reason="Never"/>
+    <disable_collisions link1="gripper_right2" link2="link1" reason="Never"/>
+    <disable_collisions link1="gripper_right2" link2="link2" reason="Never"/>
+    <disable_collisions link1="gripper_right2" link2="link3" reason="Never"/>
+    <disable_collisions link1="gripper_right2" link2="link4" reason="Never"/>
+    <disable_collisions link1="gripper_right2" link2="link5" reason="Never"/>
+    <disable_collisions link1="gripper_right2" link2="link6" reason="Never"/>
+    <disable_collisions link1="gripper_right3" link2="link1" reason="Never"/>
+    <disable_collisions link1="gripper_right3" link2="link2" reason="Never"/>
+    <disable_collisions link1="gripper_right3" link2="link3" reason="Never"/>
+    <disable_collisions link1="gripper_right3" link2="link4" reason="Never"/>
+    <disable_collisions link1="gripper_right3" link2="link5" reason="Never"/>
+    <disable_collisions link1="gripper_right3" link2="link6" reason="Never"/>
+    <disable_collisions link1="link1" link2="link2" reason="Adjacent"/>
+    <disable_collisions link1="link1" link2="link3" reason="Default"/>
+    <disable_collisions link1="link1" link2="link5" reason="Never"/>
+    <disable_collisions link1="link2" link2="link3" reason="Adjacent"/>
+    <disable_collisions link1="link2" link2="link4" reason="Never"/>
+    <disable_collisions link1="link2" link2="link5" reason="Never"/>
+    <disable_collisions link1="link3" link2="link4" reason="Adjacent"/>
+    <disable_collisions link1="link3" link2="link5" reason="Never"/>
+    <disable_collisions link1="link4" link2="link5" reason="Adjacent"/>
+    <disable_collisions link1="link5" link2="link6" reason="Adjacent"/>
 </robot>

File: urdf/mycobot_320.urdf.xacro (robot description, xacro)
@@ -1,4 +1,4 @@
 <?xml version="1.0"?>
-<robot xmlns:xacro="http://wiki.ros.org/xacro" name="$(arg name)">
+<robot xmlns:xacro="http://wiki.ros.org/xacro" name="mycobot_320">
    <!-- Robot name parameter -->
    <xacro:arg name="name" default="mycobot_320"/>
@@ -7,9 +7,9 @@
    <!-- Parameters -->
    <xacro:arg name="prefix" default="" />
-   <xacro:arg name="joint_limit_params" default=""/>
-   <xacro:arg name="kinematics_params" default=""/>
-   <xacro:arg name="physical_params" default=""/>
-   <xacro:arg name="visual_params" default=""/>
-    <!-- Simulation parameters -->
+   <xacro:arg name="joint_limit_params" default="$(find cobot_demo)/config/joint_limits.yaml"/>
+   <xacro:arg name="kinematics_params" default="$(find cobot_demo)/config/default_kinematics.yaml"/>
+   <xacro:arg name="physical_params" default="$(find cobot_demo)/config/physical_parameters.yaml"/>
+   <xacro:arg name="visual_params" default="$(find cobot_demo)/config/visual_parameters.yaml"/>
+   <!-- Simulation parameters -->
    <xacro:arg name="use_fake_hardware" default="true" />
    <!-- Initial position for fake hardware -->
@@ -33,13 +33,17 @@
    <xacro:include filename="$(find cobot_demo)/urdf/gripper_macro.xacro"/>
    <xacro:gripper></xacro:gripper>
-   <xacro:include filename="$(find cobot_demo)/urdf/gripper.ros2_control.xacro"/>
+<!--    <xacro:include filename="$(find cobot_demo)/urdf/gripper.ros2_control.xacro"/>
    <xacro:gripper_ros2_control use_fake_hardware="$(arg use_fake_hardware)">
-   </xacro:gripper_ros2_control>
-    <!-- Gripper -->
-    <!-- <link name="gripper"/> -->
-    <joint name="link6-gripper" type="fixed">
+   </xacro:gripper_ros2_control> -->
+    <joint name="link6-gripper-base" type="fixed">
+      <origin xyz="0 0 0" rpy="0 0 0"/>
+      <parent link="link6"/>
+      <child link="gripper_base"/>
+    </joint>
+    <link name="gripper"/>
+    <joint name="link6-gripper-center" type="fixed">
       <origin xyz="0 0 0.025" rpy="0 0 0"/>
       <parent link="link6"/>
-      <child link="gripper_base"/>
+      <child link="gripper"/>
     </joint>
     <!-- Camera frame -->
@@ -57,5 +61,3 @@
       <child link="target"/>
     </joint>
-    <!-- Include gripper -->
-    <xacro:include filename="$(find mycobot_320_description)/urdf/inc/mycobot_common.xacro" />
 </robot>
