Commit message: working with fake controller

File: urdf/mycobot_320.srdf.xacro (robot description, xacro)
@@ -8,5 +8,5 @@
         <joint name="joint5" />
         <joint name="joint6" />
-        <joint name="gripper_controller" />
+        <!-- <joint name="gripper_controller" /> -->
     </group>
     <group name="gripper_group">
@@ -20,5 +20,5 @@
         <joint name="joint5" value="0" />
         <joint name="joint6" value="0" />
-        <joint name="gripper_controller" value="0" />
+        <!-- <joint name="gripper_controller" value="0" /> -->
     </group_state>
     <virtual_joint name="vitual_joint" type="fixed" parent_frame="basic" child_link="base_link" />

File: urdf/mycobot_320.urdf.xacro (robot description, xacro)
@@ -33,7 +33,4 @@
    <xacro:include filename="$(find cobot_demo)/urdf/gripper_macro.xacro"/>
    <xacro:gripper></xacro:gripper>
-<!--    <xacro:include filename="$(find cobot_demo)/urdf/gripper.ros2_control.xacro"/>
-   <xacro:gripper_ros2_control use_fake_hardware="$(arg use_fake_hardware)">
-   </xacro:gripper_ros2_control> -->
     <joint name="link6-gripper-base" type="fixed">
       <origin xyz="0 0 0" rpy="0 0 0"/>
