Commit message: fixed gripper base mesh, added predefined poses

File: urdf/gripper_macro.xacro (robot description, xacro)
@@ -3,8 +3,12 @@
 <xacro:macro name="gripper">
 <xacro:property name="width" value=".2" />
+<material name="white">
+  <color rgba="1 1 1 1"/>
+</material>
   <link name="gripper_base">
     <visual>
       <geometry>
-       <mesh filename="package://cobot_demo/urdf/meshes/gripper_base.dae"/>
+       <mesh scale="0.001 0.001 0.001" filename="package://cobot_demo/urdf/meshes/collision/gripper_base.dae"/>
+       <material name="white"/>
       </geometry>
     <origin xyz = "-0.02 0.012 -0.018 " rpy = " 1.5708 0 1.5708"/>
@@ -12,5 +16,5 @@
     <collision>
       <geometry>
-       <mesh filename="package://cobot_demo/urdf/meshes/gripper_base.dae"/>
+       <mesh scale="0.001 0.001 0.001" filename="package://cobot_demo/urdf/meshes/collision/gripper_base.dae"/>
       </geometry>
     <origin xyz = "-0.02 0.012 -0.018 " rpy = " 1.5708 0 1.5708"/>

File: urdf/mycobot_320.urdf.xacro (robot description, xacro)
@@ -52,9 +52,9 @@
     </joint>
     <!-- Target frame for simulation-->
-    <link name="target"/>
+<!--     <link name="target"/>
     <joint name="base-target" type="fixed">
       <origin xyz="-0.045 -0.214 0.353" rpy="${radians(-106.984)} ${radians(-23.960)} ${radians(-172.926)}"/>
       <parent link="base_link"/>
       <child link="target"/>
-    </joint>
+    </joint> -->
 </robot>
