Commit message: wip

File: urdf/mycobot_320.urdf.xacro (robot description, xacro)
@@ -34,5 +34,5 @@
    <xacro:gripper></xacro:gripper>
     <joint name="link6-gripper-base" type="fixed">
-      <origin xyz="0 0 0" rpy="0 0 0"/>
+      <origin xyz="0 -0.01 0.06" rpy="1.5708 0 0"/>
       <parent link="link6"/>
       <child link="gripper_base"/>
@@ -40,5 +40,5 @@
     <link name="gripper"/>
     <joint name="link6-gripper-center" type="fixed">
-      <origin xyz="0 0 0.025" rpy="0 0 0"/>
+      <origin xyz="0 0 0.15" rpy="0 0 0"/>
       <parent link="link6"/>
       <child link="gripper"/>
@@ -47,12 +47,12 @@
     <link name="camera"/>
     <joint name="link6-camera" type="fixed">
-      <origin xyz="0 0 0.075" rpy="0 0 0"/>
+      <origin xyz="0 -0.0762 0" rpy="0 0 0"/>
       <parent link="link6"/>
       <child link="camera"/>
     </joint>
-    <!-- Target -->
+    <!-- Target frame for simulation-->
     <link name="target"/>
     <joint name="base-target" type="fixed">
-      <origin xyz="-0.035 -0.214 0.353" rpy="${radians(-106.984)} ${radians(-23.960)} ${radians(-172.926)}"/>
+      <origin xyz="-0.045 -0.214 0.353" rpy="${radians(-106.984)} ${radians(-23.960)} ${radians(-172.926)}"/>
       <parent link="base_link"/>
       <child link="target"/>

Commit message: updated camera frame to match new mounting position

File: urdf/mycobot_320.urdf.xacro (robot description, xacro)
@@ -47,5 +47,5 @@
     <link name="camera"/>
     <joint name="link6-camera" type="fixed">
-      <origin xyz="0 -0.0762 0" rpy="0 0 0"/>
+      <origin xyz="0.0762 0 0" rpy="0 0 0"/>
       <parent link="link6"/>
       <child link="camera"/>

Commit message: updated tf between aruco and target

File: urdf/mycobot_320.urdf.xacro (robot description, xacro)
@@ -54,7 +54,14 @@
 <!--     <link name="target"/>
     <joint name="base-target" type="fixed">
-      <origin xyz="-0.045 -0.214 0.353" rpy="${radians(-106.984)} ${radians(-23.960)} ${radians(-172.926)}"/>
+      <origin xyz="0.247 0.258 0.061" rpy="${radians(-178.566)} ${radians(-34.538)} ${radians(56.878)}"/>
       <parent link="base_link"/>
       <child link="target"/>
     </joint> -->
+    <!-- Aruco frame for simulation-->
+<!--     <link name="aruco"/>
+    <joint name="base-aruco" type="fixed">
+      <origin xyz="0.247 0.219 0.066" rpy="${radians(49.866)} ${radians(14.975)} ${radians(-32.234)}"/>
+      <parent link="base_link"/>
+      <child link="aruco"/>
+    </joint> -->
 </robot>

Commit message: added hdd caddy mesh, aruco and target frames for simulation

File: urdf/mycobot_320.urdf.xacro (robot description, xacro)
@@ -51,17 +51,41 @@
       <child link="camera"/>
     </joint>
-    <!-- Target frame for simulation-->
-<!--     <link name="target"/>
-    <joint name="base-target" type="fixed">
-      <origin xyz="0.247 0.258 0.061" rpy="${radians(-178.566)} ${radians(-34.538)} ${radians(56.878)}"/>
-      <parent link="base_link"/>
-      <child link="target"/>
-    </joint> -->
     <!-- Aruco frame for simulation-->
-<!--     <link name="aruco"/>
+    <link name="aruco"/>
     <joint name="base-aruco" type="fixed">
-      <origin xyz="0.247 0.219 0.066" rpy="${radians(49.866)} ${radians(14.975)} ${radians(-32.234)}"/>
+      <origin xyz="0.247 0.219 0.066" rpy="${radians(0)} ${radians(0)} ${radians(0)}"/>
       <parent link="base_link"/>
       <child link="aruco"/>
-    </joint> -->
+    </joint>
+    <!-- Target frame for simulation-->
+    <link name="target"/>
+    <joint name="aruco-target" type="fixed">
+      <origin xyz="0.0 0.0 0.06" rpy="${radians(-90)} ${radians(0)} ${radians(0)}"/>
+      <parent link="aruco"/>
+      <child link="target"/>
+    </joint>
+    <!-- HDD caddy for simulation-->
+    <material name="black">
+      <color rgba="0 0 0 1"/>
+    </material>
+    <link name="hdd_caddy">
+      <visual>
+        <geometry>
+         <mesh filename="package://cobot_demo/urdf/meshes/hdd_caddy.dae"/>
+         <material name="black"/>
+        </geometry>
+      <origin xyz = "0 0 0" rpy = "0 0 0"/>
+      </visual>
+      <collision>
+        <geometry>
+         <mesh filename="package://cobot_demo/urdf/meshes/hdd_caddy.dae"/>
+        </geometry>
+      <origin xyz = "0 0 0" rpy = "0 0 0"/>
+      </collision>
+    </link>
+    <joint name="aruco-hdd_caddy" type="fixed">
+      <origin xyz="0 0 0" rpy="${radians(0)} ${radians(0)} ${radians(0)}"/>
+      <parent link="aruco"/>
+      <child link="hdd_caddy"/>
+    </joint>
 </robot>

Commit message: added support for multi arucos/hard drives

File: urdf/mycobot_320.urdf.xacro (robot description, xacro)
@@ -47,45 +47,33 @@
     <link name="camera"/>
     <joint name="link6-camera" type="fixed">
-      <origin xyz="0.0762 0 0" rpy="0 0 0"/>
+      <origin xyz="0 0.04405 0.0508" rpy="0 0 0"/>
       <parent link="link6"/>
       <child link="camera"/>
     </joint>
     <!-- Aruco frame for simulation-->
-    <link name="aruco"/>
-    <joint name="base-aruco" type="fixed">
-      <origin xyz="0.247 0.219 0.066" rpy="${radians(0)} ${radians(0)} ${radians(0)}"/>
+    <link name="aruco_36"/> <!-- Large drive-->
+    <joint name="base-aruco-36" type="fixed">
+      <origin xyz="0.176 -0.344 0.124" rpy="${radians(0.361)} ${radians(1.711)} ${radians(-126.413)}"/>
       <parent link="base_link"/>
-      <child link="aruco"/>
+      <child link="aruco_36"/>
+    </joint>
+    <link name="aruco_165"/> <!-- Small drive-->
+    <joint name="base-aruco-165" type="fixed">
+      <origin xyz="0.267 0.219 0.066" rpy="${radians(0)} ${radians(0)} ${radians(0)}"/>
+      <parent link="base_link"/>
+      <child link="aruco_165"/>
     </joint>
     <!-- Target frame for simulation-->
-    <link name="target"/>
-    <joint name="aruco-target" type="fixed">
+    <link name="large_drive"/>
+    <joint name="aruco-large_drive" type="fixed">
+      <origin xyz="0.0 0.085 0.06" rpy="${radians(-90)} ${radians(0)} ${radians(0)}"/>
+      <parent link="aruco_36"/>
+      <child link="large_drive"/>
+    </joint>
+    <link name="small_drive"/>
+    <joint name="aruco-small_drive" type="fixed">
       <origin xyz="0.0 0.0 0.06" rpy="${radians(-90)} ${radians(0)} ${radians(0)}"/>
-      <parent link="aruco"/>
-      <child link="target"/>
-    </joint>
-    <!-- HDD caddy for simulation-->
-    <material name="black">
-      <color rgba="0 0 0 1"/>
-    </material>
-    <link name="hdd_caddy">
-      <visual>
-        <geometry>
-         <mesh filename="package://cobot_demo/urdf/meshes/hdd_caddy.dae"/>
-         <material name="black"/>
-        </geometry>
-      <origin xyz = "0 0 0" rpy = "0 0 0"/>
-      </visual>
-      <collision>
-        <geometry>
-         <mesh filename="package://cobot_demo/urdf/meshes/hdd_caddy.dae"/>
-        </geometry>
-      <origin xyz = "0 0 0" rpy = "0 0 0"/>
-      </collision>
-    </link>
-    <joint name="aruco-hdd_caddy" type="fixed">
-      <origin xyz="0 0 0" rpy="${radians(0)} ${radians(0)} ${radians(0)}"/>
-      <parent link="aruco"/>
-      <child link="hdd_caddy"/>
+      <parent link="aruco_165"/>
+      <child link="small_drive"/>
     </joint>
 </robot>

Commit message: fixed bug with joint slider update to match joint state, fixed hdd holder dimensions

File: urdf/mycobot_320.urdf.xacro (robot description, xacro)
@@ -54,5 +54,5 @@
     <link name="aruco_36"/> <!-- Large drive-->
     <joint name="base-aruco-36" type="fixed">
-      <origin xyz="0.176 -0.344 0.124" rpy="${radians(0.361)} ${radians(1.711)} ${radians(-126.413)}"/>
+      <origin xyz="0.142 -0.249 0.046" rpy="${radians(5.040)} ${radians(1.109)} ${radians(-119.986)}"/>
       <parent link="base_link"/>
       <child link="aruco_36"/>

Commit message: added target approach pose

File: urdf/mycobot_320.urdf.xacro (robot description, xacro)
@@ -71,4 +71,10 @@
       <child link="large_drive"/>
     </joint>
+    <link name="large_drive_approach"/>
+    <joint name="large_drive-approach" type="fixed">
+      <origin xyz="0.0 0.0 -0.03" rpy="${radians(0)} ${radians(0)} ${radians(0)}"/>
+      <parent link="large_drive"/>
+      <child link="large_drive_approach"/>
+    </joint>
     <link name="small_drive"/>
     <joint name="aruco-small_drive" type="fixed">

Commit message: wip

File: urdf/mycobot_320.urdf.xacro (robot description, xacro)
@@ -51,6 +51,6 @@
       <child link="camera"/>
     </joint>
-    <!-- Aruco frame for simulation-->
-    <link name="aruco_36"/> <!-- Large drive-->
+    <!-- Frames for simulation-->
+<!--     <link name="aruco_36"/>
     <joint name="base-aruco-36" type="fixed">
       <origin xyz="0.142 -0.249 0.046" rpy="${radians(5.040)} ${radians(1.109)} ${radians(-119.986)}"/>
@@ -58,5 +58,5 @@
       <child link="aruco_36"/>
     </joint>
-    <link name="aruco_165"/> <!-- Small drive-->
+    <link name="aruco_165"/>
     <joint name="base-aruco-165" type="fixed">
       <origin xyz="0.267 0.219 0.066" rpy="${radians(0)} ${radians(0)} ${radians(0)}"/>
@@ -64,5 +64,4 @@
       <child link="aruco_165"/>
     </joint>
-    <!-- Target frame for simulation-->
     <link name="large_drive"/>
     <joint name="aruco-large_drive" type="fixed">
@@ -77,4 +76,10 @@
       <child link="large_drive_approach"/>
     </joint>
+    <link name="large_drive_retract"/>
+    <joint name="large_drive-retract" type="fixed">
+      <origin xyz="0.0 -0.05 0.0" rpy="${radians(0)} ${radians(0)} ${radians(0)}"/>
+      <parent link="large_drive"/>
+      <child link="large_drive_retract"/>
+    </joint>
     <link name="small_drive"/>
     <joint name="aruco-small_drive" type="fixed">
@@ -82,4 +87,4 @@
       <parent link="aruco_165"/>
       <child link="small_drive"/>
-    </joint>
+    </joint> -->
 </robot>
